File: hardware/kicad/generated/thumbdeck_left.kicad_pcb (KiCad board)
At the start: 4 copper layers, 79.5 x 97 mm, 85 parts, among them J2 FFC16, SW1 SNAP7, SW10 SNAP7, SW11 SNAP7, SW12 SNAP7, SW13 SNAP7, SW14 SNAP7, SW15 SNAP7, SW16 SNAP7, SW17 SNAP7, SW18 SNAP7, SW19 SNAP7, SW2 SNAP7, SW20 SNAP7, SW21 SNAP7, SW22 SNAP7, SW23 SNAP7, SW24 SNAP7, SW25 SNAP7, SW26 SNAP7, SW27 SNAP7, SW28 SNAP7, SW29 SNAP7, SW3 SNAP7, SW30 SNAP7, SW31 SNAP7, SW32 SNAP7, SW33 SNAP7, SW34 SNAP7, SW35 SNAP7, SW36 SNAP7, SW37 SNAP7, SW38 SNAP7, SW39 SNAP7, SW4 SNAP7, SW40 SNAP7, SW41 SNAP7, SW42 SNAP7, SW5 SNAP7, SW6 SNAP7, SW7 SNAP7, SW8 SNAP7, SW9 SNAP7

Commit message: fixed keybaord issues
Parts:
- moved D39 21.4 mm to (34.2, 15.0)
- moved SW39 21.4 mm to (34.2, 18.0)
- moved D40 12.6 mm to (51.2, 15.0)
- moved SW40 12.6 mm to (51.2, 18.0)
- moved D10 4.49 mm to (32.8, 45.5)
- moved D14 4.49 mm to (52.8, 54.5)
- moved D15 4.49 mm to (42.8, 54.5)
- moved D16 4.49 mm to (32.8, 54.5)
- moved D2 4.49 mm to (52.8, 36.5)
- moved D20 4.49 mm to (52.8, 63.5)
- moved D21 4.49 mm to (42.8, 63.5)
- moved D22 4.49 mm to (32.8, 63.5)
- moved D26 4.49 mm to (52.8, 72.5)
- moved D27 4.49 mm to (42.8, 72.5)
- moved D28 4.49 mm to (32.8, 72.5)
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Routing:
- net COL8: track 186.2 -> 167.0 mm, vias 4 -> 3
- net COL9: track 182.1 -> 195.2 mm, vias 2 -> 4
- net ROW8: track 93.5 -> 99.5 mm
- net ROW7: track 102.0 -> 96.2 mm, vias 0 -> 2
- net DN_L29: track 17.0 -> 22.2 mm
- net COL5: track 216.7 -> 214.0 mm, vias 3 -> 5
- net COL6: track 224.8 -> 227.5 mm
- net DN_L34: track 17.2 -> 19.4 mm
- net DN_L2: track 17.7 -> 20.0 mm
- net DN_L5: track 20.7 -> 19.1 mm
- net DN_L25: track 16.9 -> 18.5 mm
- net DN_L3: track 20.1 -> 18.6 mm
- net DN_L35: track 17.1 -> 18.5 mm
- net DN_L23: track 16.6 -> 17.6 mm
- net COL7: track 170.6 -> 171.5 mm
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Other:
- board size 79.5 x 97 mm -> 75 x 98 mm
