File: hardware/kicad/generated/thumbdeck_left.kicad_pcb (KiCad board)
At the start: 4 copper layers, 75 x 98 mm, 85 parts, among them J2 FFC16, SW1 SNAP7, SW10 SNAP7, SW11 SNAP7, SW12 SNAP7, SW13 SNAP7, SW14 SNAP7, SW15 SNAP7, SW16 SNAP7, SW17 SNAP7, SW18 SNAP7, SW19 SNAP7, SW2 SNAP7, SW20 SNAP7, SW21 SNAP7, SW22 SNAP7, SW23 SNAP7, SW24 SNAP7, SW25 SNAP7, SW26 SNAP7, SW27 SNAP7, SW28 SNAP7, SW29 SNAP7, SW3 SNAP7, SW30 SNAP7, SW31 SNAP7, SW32 SNAP7, SW33 SNAP7, SW34 SNAP7, SW35 SNAP7, SW36 SNAP7, SW37 SNAP7, SW38 SNAP7, SW39 SNAP7, SW4 SNAP7, SW40 SNAP7, SW41 SNAP7, SW42 SNAP7, SW5 SNAP7, SW6 SNAP7, SW7 SNAP7, SW8 SNAP7, SW9 SNAP7

Commit message: added typing screen
Parts:
- added F1: PPTC-0.75A, Fuse_1812_4532Metric, B.Cu at (50.0, 91.5)
- added J4: JST-PH-2, JST_PH_S2B-PH-SM4-TB_1x02-1MP_P2.00mm_Horizontal, B.Cu at (60.0, 91.5)
- J2: value FFC16 -> FFC20; footprint ffc_afa07_s16fcc -> ffc_afa07_s20fcc
- moved J2 4.00 mm to (71.4, 68.5), turned to -90 degrees
Connections:
- J2 pad 10: ROW6 -> ROW7
- J2 pad 11: ROW5 -> ROW8
- J2 pad 12: ROW4 -> COL5
- J2 pad 13: ROW3 -> COL6
- J2 pad 14: ROW2 -> COL7
- J2 pad 15: ROW1 -> COL8
- J2 pad 16: ROW0 -> COL9
- J2 pad 3: COL9 -> ROW0
- J2 pad 4: COL8 -> ROW1
- J2 pad 5: COL7 -> ROW2
- J2 pad 6: COL6 -> ROW3
- J2 pad 7: COL5 -> ROW4
- J2 pad 8: ROW8 -> ROW5
- J2 pad 9: ROW7 -> ROW6
Routing:
- net COL5: track 223.5 -> 0.00 mm, vias 7 -> 0
- net COL6: track 216.4 -> 0.00 mm, vias 2 -> 0
- net COL9: track 194.4 -> 0.00 mm, vias 4 -> 0
- net COL8: track 175.4 -> 0.00 mm, vias 2 -> 0
- net COL7: track 170.7 -> 0.00 mm, vias 2 -> 0
- net ROW7: track 96.2 -> 0.00 mm, vias 2 -> 0
- net ROW8: track 93.7 -> 0.00 mm, vias 2 -> 0
- net ROW1: track 81.0 -> 0.00 mm
- net ROW0: track 75.8 -> 0.00 mm
- net ROW2: track 72.7 -> 0.00 mm
- net ROW3: track 66.8 -> 0.00 mm
- net ROW6: track 66.7 -> 0.00 mm
- net ROW4: track 66.3 -> 0.00 mm
- net ROW5: track 62.7 -> 0.00 mm
- net DN_L6: track 19.6 -> 0.00 mm, vias 1 -> 0
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Other:
- outline, holes or cut-outs redrawn
- board text added: "+"
- board text added: "-"
- board text added: "20P TYPE-A"
- board text added: "BAT"
- board text added: "F1 PPTC 0.75A"
- board text removed: "J2 FFC16 <- pin1"
