File: hardware/kicad/generated/thumbdeck_right.kicad_pcb (KiCad board)
At the start: 4 copper layers, 79.5 x 97 mm, 111 parts, among them J1 USB-C, J2 FFC16, J3 JST-PH-2, SW1 SNAP7, SW10 SNAP7, SW11 SNAP7, SW12 SNAP7, SW13 SNAP7, SW14 SNAP7, SW15 SNAP7, SW16 SNAP7, SW17 SNAP7, SW18 SNAP7, SW19 SNAP7, SW2 SNAP7, SW20 SNAP7, SW21 SNAP7, SW22 SNAP7, SW23 SNAP7, SW24 SNAP7, SW25 SNAP7, SW26 SNAP7, SW27 SNAP7, SW28 SNAP7, SW29 SNAP7, SW3 SNAP7, SW30 SNAP7, SW31 SNAP7, SW32 SNAP7, SW33 SNAP7, SW34 SNAP7, SW35 SNAP7, SW36 SNAP7, SW4 SNAP7, SW5 SNAP7, SW6 SNAP7, SW7 SNAP7, SW8 SNAP7, SW9 SNAP7, SW90 MSK12C02, SW91 TS-1187A, U1 E73-2G4M08S1C, U2 MCP73831, U3 USBLC6-2SC6

Commit message: fixed keybaord issues
Routing:
- net COL7: track 97.0 -> 128.7 mm
- net VBAT_CELL: track 144.8 -> 121.4 mm
- net COL2: track 185.4 -> 170.6 mm
- net DN_R31: track 29.8 -> 17.1 mm
- net TP_INT: track 35.8 -> 24.3 mm
- net VBUS: track 60.4 -> 49.7 mm, vias 2 -> 4
- net ROW4: track 154.2 -> 143.4 mm
- net SWDCLK: track 28.7 -> 38.6 mm
- net COL1: track 157.7 -> 166.6 mm, vias 4 -> 3
- net VBAT_SENSE: track 8.47 -> 17.4 mm, vias 0 -> 2
- net COL0: track 196.9 -> 188.3 mm, vias 3 -> 5
- net COL6: track 121.4 -> 128.1 mm
- net ROW0: track 137.3 -> 131.0 mm, vias 2 -> 4
- net COL5: track 108.7 -> 103.0 mm, vias 3 -> 2
- net USB_DM: track 48.2 -> 42.7 mm
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Other:
- board size 79.5 x 97 mm -> 75 x 98 mm
