File: hardware/kicad/generated/thumbdeck_right.kicad_pcb (KiCad board)
At the start: 4 copper layers, 75 x 98 mm, 111 parts, among them J1 USB-C, J2 FFC16, J3 JST-PH-2, SW1 SNAP7, SW10 SNAP7, SW11 SNAP7, SW12 SNAP7, SW13 SNAP7, SW14 SNAP7, SW15 SNAP7, SW16 SNAP7, SW17 SNAP7, SW18 SNAP7, SW19 SNAP7, SW2 SNAP7, SW20 SNAP7, SW21 SNAP7, SW22 SNAP7, SW23 SNAP7, SW24 SNAP7, SW25 SNAP7, SW26 SNAP7, SW27 SNAP7, SW28 SNAP7, SW29 SNAP7, SW3 SNAP7, SW30 SNAP7, SW31 SNAP7, SW32 SNAP7, SW33 SNAP7, SW34 SNAP7, SW35 SNAP7, SW36 SNAP7, SW4 SNAP7, SW5 SNAP7, SW6 SNAP7, SW7 SNAP7, SW8 SNAP7, SW9 SNAP7, SW90 MSK12C02, SW91 TS-1187A, U1 E73-2G4M08S1C, U2 MCP73831, U3 USBLC6-2SC6

Commit message: v0.21: right-grip ThinkPad-style pointing nub — Bean-architecture TMAG5273 hall sensor
The right top zone mirrors the left cluster: PgUp/PgDn at the mouse-button
mirror, and a rate-control pointing nub at the exact D-pad mirror (32.3, 79.0).
Architecture per the Ploopy Bean (CERN-OHL-S v2, credited): a TMAG5273A1 I2C
hall sensor (C3716049, SOT-23-6, machine-placed SMT on the back) reads a
O4x2 N52 magnet in a printed flexure spring through the 1.6mm FR4; firmware
maps deflection to cursor VELOCITY (quadratic curve + deadzone + remainder).
An ALPS RKJXV gimbal variant was fully implemented first and rejected — the
11.2mm module body protruded through the face; recorded in the design log.

- board: U4 + R26/R27 pullups + C8 on the reserved TP6-8 I2C nets (P0.05/28/29),
  all-SMT again (71/43 placements); reworked USB In2 lane elbow; pre-placed GND
  escapes for U1.21/24 (fan-out walled their pour blob in deterministically);
  both boards routed 0 violations / 0 unconnected
- firmware: in-tree Zephyr module tmag5273_nub (Apache-2.0, register map from
  the upstream Zephyr driver, NOT the Bean's GPL QMK): 100Hz poll, boot zero
  calibration, DT-tunable curve, pm_device sleep hook (continuous mode would
  drain ~2.3mA through ZMK deep sleep); matrix stays 78 keys
- CAD: flat face with a O10 aperture; prints 8+9 = nub_spring (flange + spiral
  arms + legs clamped by the lid counterbore at 0.05 preload) and TPU nub_cap
  (4.25mm proud); 221 bodies, 0 collisions; GLB includes the nub
- docs: BOM/assembly/README/design-log rewritten for the nub; magnet polarity
  procedure; CI marked stale pending a v0.21 re-run; 78-key counts restored
- verified by a 17-agent adversarial review: fixed the spigot z-stack (cap had
  0.15mm engagement), the unclamped spring flange, and the sensor sleep drain

Co-Authored-By: Claude Fable 5 <noreply@anthropic.com>
Parts:
- added C8: 100nF, C_0402_1005Metric, B.Cu at (32.3, 24.0)
- added R26: 4k7, R_0402_1005Metric, B.Cu at (36.0, 28.5)
- added R27: 4k7, R_0402_1005Metric, B.Cu at (38.5, 28.5)
- added U4: TMAG5273, SOT-23-6, B.Cu at (32.3, 18.0)
- moved D35 35.2 mm to (45.7, 9.50)
- moved D36 35.2 mm to (45.7, 20.5)
- moved SW35 35.2 mm to (45.7, 12.5)
- moved SW36 35.2 mm to (45.7, 23.5)
- moved SW91 18.6 mm to (53.5, 25.5)
- moved C7 10.4 mm to (47.5, 3.50)
- moved TP6 8.21 mm to (48.0, 29.5)
- moved TP7 8.21 mm to (45.5, 29.5)
- moved TP8 8.21 mm to (43.0, 29.5)
Routing:
- net 3V3: track 7.11 -> 52.6 mm, vias 0 -> 4
- net SCL: track 29.1 -> 69.9 mm, vias 2 -> 0
- net COL4: track 171.0 -> 135.2 mm, vias 2 -> 1
- net VBUS: track 49.7 -> 79.5 mm, vias 4 -> 3
- net SDA: track 16.2 -> 42.8 mm
- net TP_INT: track 24.3 -> 48.2 mm, vias 2 -> 3
- net RESET: track 30.6 -> 18.1 mm
- net COL7: track 128.7 -> 116.2 mm
- net ROW6: track 196.1 -> 183.9 mm
- net COL6: track 128.1 -> 116.3 mm
- net ROW7: track 114.4 -> 103.0 mm, vias 2 -> 4
- net VBAT_CELL: track 121.4 -> 110.0 mm
- net USB_DP: track 61.8 -> 50.9 mm, vias 4 -> 3
- net SWDCLK: track 38.6 -> 28.6 mm
- net ROW8: track 102.2 -> 111.3 mm
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
Commit message: v0.22: true-mirror page keys + genuine-TrackPoint-cap nub mount
Two feedback items on the v0.21 print:

- PGUP/PGDN move to the TRUE mouse-button mirror x=57.25 (the F10|DEL gap,
  mirroring the left pair's ESC|F1 gap; was 45.7, "above F9"). v0.21's
  blocker was a face-conflation: domes are front-side, the E73 is back-side —
  they coexist. Both feature diodes drop to deck y73.2 under the TP row
  (defaults hit the module belly / the SWD row), SW91 moves to the vacated
  old-PGUP zone (46.0, 80.5). Both boards re-route 0/0 on the first 40-pass
  attempt; fab re-exported (71/43); sim 78 keys PASS; firmware byte-identical.
- The nub becomes compatible with genuine ThinkPad caps: the spring's post is
  the classic-cap standard 4.4mm-square x 2.5 platform (classic full-size
  caps: ~4.5mm square socket, dims cross-checked against navcaps' printed
  cap mounts), and the printed cap is a classic soft-dome replica in
  ThinkPad-RED TPU (O7.8 mushroom, dot grid, same socket) — printed and
  genuine caps interchange. Hub top drops to z14.0 so the cap skirt nestles
  into the O10 aperture like a real TrackPoint; first tilt-stop is now the
  rubber skirt (gentler on the flexure). GLB paints it trackpoint_red.
- verify_alignment.py taught the v0.22 topology (DIODE_DECK overrides +
  side-aware courtyard check) — gate back to ALL CHECKS PASS.
- Adversarial review (13 agents) fixes folded in: cap waist O6.2->O6.8 (the
  socket corner left a 0.10mm unprintable wall at the waist — now 0.40mm),
  stale intermediate coordinates in the design log, stale doc claims.

Co-Authored-By: Claude Fable 5 <noreply@anthropic.com>
Parts:
- moved D35 15.8 mm to (52.5, 23.8)
- moved D36 12.0 mm to (57.2, 23.8)
- moved SW91 11.7 mm to (46.0, 16.5)
- moved SW35 11.5 mm to (57.2, 12.5)
- moved SW36 11.5 mm to (57.2, 23.5)
Routing:
- net ROW7: track 103.0 -> 156.5 mm
- net VBAT: track 74.5 -> 102.4 mm
- net SWDCLK: track 28.6 -> 42.0 mm
- net ROW4: track 152.4 -> 165.4 mm, vias 4 -> 2
- net COL8: track 119.5 -> 132.3 mm
- net COL9: track 102.4 -> 114.7 mm
- net SCL: track 69.9 -> 57.8 mm, vias 0 -> 3
- net DN_R35: track 18.4 -> 30.4 mm
- net COL0: track 180.1 -> 192.1 mm, vias 4 -> 3
- net COL7: track 116.2 -> 104.9 mm
- net ROW3: track 146.1 -> 154.9 mm, vias 4 -> 2
- net ROW6: track 183.9 -> 175.3 mm
- net VBUS: track 79.5 -> 71.3 mm, vias 3 -> 2
- net ROW1: track 141.5 -> 149.6 mm, vias 2 -> 5
- net COL3: track 179.9 -> 173.7 mm
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