File: hardware/kicad/generated/thumbdeck_right.kicad_pcb (KiCad board)
At the start: 4 copper layers, 75 x 98 mm, 115 parts, among them J1 USB-C, J2 FFC16, J3 JST-PH-2, SW1 SNAP7, SW10 SNAP7, SW11 SNAP7, SW12 SNAP7, SW13 SNAP7, SW14 SNAP7, SW15 SNAP7, SW16 SNAP7, SW17 SNAP7, SW18 SNAP7, SW19 SNAP7, SW2 SNAP7, SW20 SNAP7, SW21 SNAP7, SW22 SNAP7, SW23 SNAP7, SW24 SNAP7, SW25 SNAP7, SW26 SNAP7, SW27 SNAP7, SW28 SNAP7, SW29 SNAP7, SW3 SNAP7, SW30 SNAP7, SW31 SNAP7, SW32 SNAP7, SW33 SNAP7, SW34 SNAP7, SW35 SNAP7, SW36 SNAP7, SW4 SNAP7, SW5 SNAP7, SW6 SNAP7, SW7 SNAP7, SW8 SNAP7, SW9 SNAP7, SW90 MSK12C02, SW91 TS-1187A, U1 E73-2G4M08S1C, U2 MCP73831, U3 USBLC6-2SC6, U4 TMAG5273

Commit message: added typing screen
Parts:
- removed J3: JST-PH-2, JST_PH_S2B-PH-SM4-TB_1x02-1MP_P2.00mm_Horizontal
- J2: value FFC16 -> FFC20; footprint ffc_afa07_s16fcc -> ffc_afa07_s20fcc
- moved J2 4.00 mm to (3.60, 68.5), turned to 90 degrees
Connections:
- J2 pad 1: ROW0 -> (no net)
- J2 pad 10: COL5 -> ROW8
- J2 pad 11: COL6 -> ROW7
- J2 pad 12: COL7 -> ROW6
- J2 pad 13: COL8 -> ROW5
- J2 pad 14: COL9 -> ROW4
- J2 pad 15: GND -> ROW3
- J2 pad 16: GND -> ROW2
- J2 pad 2: ROW1 -> VBAT_CELL
- J2 pad 3: ROW2 -> VBAT_CELL
- J2 pad 4: ROW3 -> (no net)
- J2 pad 5: ROW4 -> COL9
- J2 pad 6: ROW5 -> COL8
- J2 pad 7: ROW6 -> COL7
- J2 pad 8: ROW7 -> COL6
- J2 pad 9: ROW8 -> COL5
Routing:
- net COL0: track 192.1 -> 0.00 mm, vias 3 -> 0
- net COL2: track 179.8 -> 0.00 mm, vias 4 -> 0
- net COL1: track 178.9 -> 0.00 mm, vias 3 -> 0
- net ROW5: track 178.6 -> 0.00 mm, vias 4 -> 0
- net ROW6: track 175.3 -> 0.00 mm, vias 5 -> 0
- net COL3: track 173.7 -> 0.00 mm, vias 3 -> 0
- net ROW4: track 165.4 -> 0.00 mm, vias 2 -> 0
- net ROW7: track 156.5 -> 0.00 mm, vias 4 -> 0
- net ROW3: track 154.9 -> 0.00 mm, vias 2 -> 0
- net ROW1: track 149.6 -> 0.00 mm, vias 5 -> 0
- net ROW2: track 147.7 -> 0.00 mm, vias 4 -> 0
- net ROW0: track 135.5 -> 0.00 mm, vias 5 -> 0
- net COL8: track 132.3 -> 0.00 mm, vias 2 -> 0
- net COL4: track 131.4 -> 0.00 mm, vias 1 -> 0
- net COL6: track 115.1 -> 0.00 mm, vias 2 -> 0
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Other:
- outline, holes or cut-outs redrawn
- board text added: "20P TYPE-A"
- board text removed: "+"
- board text removed: "-"
- board text removed: "BAT"
- board text removed: "J2 FFC16 <- pin1"
